Commit message: [ADD and EDIT]: Implementing the Launch of Hexacopter in Gazebo

File: ros_ws/src/hexacopter_description/urdf/variable_tilt_hexacopter.urdf.xacro (robot description, xacro)
@@ -5,10 +5,10 @@
   ====================== -->
   <!-- Base Dimensions and Parameters -->
-  <xacro:property name="base_mass"    value="4.253"/>
-  <xacro:property name="base_ixx"     value="0.1174"/>
-  <xacro:property name="base_iyy"     value="0.2322"/>
-  <xacro:property name="base_izz"     value="4.253"/>
+  <xacro:property name="base_mass"    value="1.5640"/>
+  <xacro:property name="base_ixx"     value="0.1"/>
+  <xacro:property name="base_iyy"     value="0.1"/>
+  <xacro:property name="base_izz"     value="0.1"/>
   <xacro:property name="base_radius"  value="0.071"/>
-  <xacro:property name="base_length"  value="0.025"/>
+  <xacro:property name="base_length"  value="0.050"/>
   <!-- Base Link -->
   <link name="base">
@@ -33,5 +33,4 @@
        2. Landing Gear
   ====================== -->
-  <!-- Properties for gear leg and skid dimensions -->
   <xacro:property name="gear_leg_length"      value="0.1"/>
   <xacro:property name="gear_leg_radius"      value="0.01"/>
@@ -39,5 +38,4 @@
   <xacro:property name="gear_skid_width"      value="0.02"/>
   <xacro:property name="gear_skid_thickness"  value="0.01"/>
-  <!-- Macro: one vertical leg + one horizontal skid -->
   <xacro:macro name="landing_gear" params="gear_name x y">
     <!-- Vertical leg link -->
@@ -45,5 +43,4 @@
       <inertial>
         <mass value="0.1"/>
-        <!-- Center of mass at mid-height of the leg -->
         <origin xyz="0 0 -${gear_leg_length/2}"/>
         <inertia ixx="0.0001" iyy="0.0001" izz="0.0001"
@@ -66,6 +63,4 @@
       <parent link="base"/>
       <child link="gear_leg_${gear_name}"/>
-      <!-- Attaching the leg to the base at (x, y, 0).
-           Adjust Z here if you want the gear further below or above the base. -->
       <origin xyz="${x} ${y} 0"/>
     </joint>
@@ -79,5 +74,4 @@
       </inertial>
       <visual>
-        <!-- Place the skid at the bottom of the leg (Z offset = -gear_leg_length) -->
         <origin xyz="0 0 -${gear_leg_length}"/>
         <geometry>
@@ -104,16 +98,21 @@
        3. Arm + Motor Properties
   ====================== -->
-  <!-- Arm Properties -->
-  <xacro:property name="arm_mass"    value="4.253"/>
-  <xacro:property name="arm_ixx"     value="0.1174"/>
-  <xacro:property name="arm_iyy"     value="0.2322"/>
-  <xacro:property name="arm_izz"     value="4.253"/>
+  <xacro:property name="arm_mass"    value="0.16"/>
+  <xacro:property name="arm_ixx"     value="0.01"/>
+  <xacro:property name="arm_iyy"     value="0.01"/>
+  <xacro:property name="arm_izz"     value="0.01"/>
   <xacro:property name="arm_length"  value="0.229"/>
-  <xacro:property name="arm_radius"  value="0.01"/>
-  <!-- Motor Properties -->
+  <xacro:property name="arm_radius"  value="0.02"/>
+  <xacro:property name="motor_mass" value="0.0880"/>
+  <xacro:property name="motor_ixx"  value="0.01"/>
+  <xacro:property name="motor_iyy"  value="0.01"/>
+  <xacro:property name="motor_izz"  value="0.01"/>
   <xacro:property name="motor_radius" value="0.02"/>
-  <xacro:property name="motor_height" value="0.02"/>
-  <!-- Propeller Properties -->
-  <xacro:property name="prop_box_length"    value="0.3"/>
+  <xacro:property name="motor_height" value="0.05"/>
+  <xacro:property name="prop_box_mass"    value="0.0240"/>
+  <xacro:property name="prop_box_ixx"     value="0.01"/>
+  <xacro:property name="prop_box_iyy"     value="0.01"/>
+  <xacro:property name="prop_box_izz"     value="0.01"/>
+  <xacro:property name="prop_box_length"    value="0.225"/>
   <xacro:property name="prop_box_width"     value="0.02"/>
   <xacro:property name="prop_box_thickness" value="0.01"/>
@@ -143,10 +142,20 @@
       </collision>
     </link>
-    <joint name="joint_arm_${arm_name}" type="fixed">
+    <!-- Revolute joint to allow arm to rotate for tilt -->
+    <joint name="joint_arm_${arm_name}" type="revolute">
       <parent link="base"/>
       <child link="arm_${arm_name}"/>
       <origin xyz="${x} ${y} ${z}" rpy="${rpy}"/>
-    </joint>
+      <axis xyz="1 0 0"/>
+      <limit lower="-1.57" upper="1.57" effort="5" velocity="2.0"/>
+    </joint>
+    <!-- Motor (Fixed to Arm) -->
     <link name="motor_${arm_name}">
+      <inertial>
+        <mass value="${motor_mass}"/>
+        <origin xyz="0 0 0"/>
+        <inertia ixx="${motor_ixx}" iyy="${motor_iyy}" izz="${motor_izz}"
+                 ixy="0" ixz="0" iyz="0"/>
+      </inertial>
       <visual>
         <origin xyz="0 0 0"/>
@@ -162,10 +171,9 @@
       </collision>
     </link>
-    <joint name="joint_motor_${arm_name}" type="revolute">
+    <!-- Fixed motor joint (no rotation with arm) -->
+    <joint name="joint_motor_${arm_name}" type="fixed">
       <parent link="arm_${arm_name}"/>
       <child link="motor_${arm_name}"/>
       <origin xyz="${arm_length/2 - motor_radius} 0 ${arm_radius}"/>
-      <axis xyz="1 0 0"/>
-      <limit lower="-1.57" upper="1.57" effort="5" velocity="2.0"/>
     </joint>
   </xacro:macro>
@@ -175,4 +183,10 @@
   <xacro:macro name="propeller" params="prop_name motor_link">
     <link name="prop_${prop_name}">
+      <inertial>
+        <mass value="${prop_box_mass}"/>
+        <origin xyz="0 0 ${prop_offset_z}"/>
+        <inertia ixx="${prop_box_ixx}" iyy="${prop_box_iyy}" izz="${prop_box_izz}"
+                 ixy="0" ixz="0" iyz="0"/>
+      </inertial>
       <visual>
         <origin xyz="0 0 ${prop_offset_z}"/>

Commit message: [EDIT]: Updating the MoI of the Hexacopter

File: ros_ws/src/hexacopter_description/urdf/variable_tilt_hexacopter.urdf.xacro (robot description, xacro)
@@ -6,7 +6,7 @@
   <!-- Base Dimensions and Parameters -->
   <xacro:property name="base_mass"    value="1.5640"/>
-  <xacro:property name="base_ixx"     value="0.1"/>
-  <xacro:property name="base_iyy"     value="0.1"/>
-  <xacro:property name="base_izz"     value="0.1"/>
+  <xacro:property name="base_ixx"     value="0.00229686"/>
+  <xacro:property name="base_iyy"     value="0.00229686"/>
+  <xacro:property name="base_izz"     value="0.00394206"/>
   <xacro:property name="base_radius"  value="0.071"/>
   <xacro:property name="base_length"  value="0.050"/>
@@ -33,6 +33,14 @@
        2. Landing Gear
   ====================== -->
-  <xacro:property name="gear_leg_length"      value="0.1"/>
-  <xacro:property name="gear_leg_radius"      value="0.01"/>
+  <xacro:property name="gear_leg_mass"    value="0.1"/>
+  <xacro:property name="gear_leg_ixx"     value="0.0001"/>
+  <xacro:property name="gear_leg_iyy"     value="0.0001"/>
+  <xacro:property name="gear_leg_izz"     value="0.0001"/>
+  <xacro:property name="gear_leg_length"  value="0.1"/>
+  <xacro:property name="gear_leg_radius"  value="0.01"/>
+  <xacro:property name="gear_skid_mass"       value="0.1"/>
+  <xacro:property name="gear_skid_ixx"        value="0.0001"/>
+  <xacro:property name="gear_skid_iyy"        value="0.0001"/>
+  <xacro:property name="gear_skid_izz"        value="0.0001"/>
   <xacro:property name="gear_skid_length"     value="0.3"/>
   <xacro:property name="gear_skid_width"      value="0.02"/>
@@ -42,7 +50,7 @@
     <link name="gear_leg_${gear_name}">
       <inertial>
-        <mass value="0.1"/>
+        <mass value="${gear_leg_mass}"/>
         <origin xyz="0 0 -${gear_leg_length/2}"/>
-        <inertia ixx="0.0001" iyy="0.0001" izz="0.0001"
+        <inertia ixx="${gear_leg_ixx}" iyy="${gear_leg_iyy}" izz="${gear_leg_izz}"
                  ixy="0" ixz="0" iyz="0"/>
       </inertial>
@@ -68,7 +76,7 @@
     <link name="gear_skid_${gear_name}">
       <inertial>
-        <mass value="0.1"/>
-        <origin xyz="0 0 0"/>
-        <inertia ixx="0.0001" iyy="0.0001" izz="0.0001"
+        <mass value="${gear_skid_mass}"/>
+        <origin xyz="0 0 0"/>
+        <inertia ixx="${gear_skid_ixx}" iyy="${gear_skid_iyy}" izz="${gear_skid_izz}"
                  ixy="0" ixz="0" iyz="0"/>
       </inertial>
@@ -99,19 +107,19 @@
   ====================== -->
   <xacro:property name="arm_mass"    value="0.16"/>
-  <xacro:property name="arm_ixx"     value="0.01"/>
-  <xacro:property name="arm_iyy"     value="0.01"/>
-  <xacro:property name="arm_izz"     value="0.01"/>
+  <xacro:property name="arm_ixx"     value="0.000715213"/>
+  <xacro:property name="arm_iyy"     value="0.000715213"/>
+  <xacro:property name="arm_izz"     value="0.000032"/>
   <xacro:property name="arm_length"  value="0.229"/>
   <xacro:property name="arm_radius"  value="0.02"/>
   <xacro:property name="motor_mass" value="0.0880"/>
-  <xacro:property name="motor_ixx"  value="0.01"/>
-  <xacro:property name="motor_iyy"  value="0.01"/>
-  <xacro:property name="motor_izz"  value="0.01"/>
+  <xacro:property name="motor_ixx"  value="0.000112917"/>
+  <xacro:property name="motor_iyy"  value="0.000112917"/>
+  <xacro:property name="motor_izz"  value="0.0000625"/>
   <xacro:property name="motor_radius" value="0.02"/>
   <xacro:property name="motor_height" value="0.05"/>
   <xacro:property name="prop_box_mass"    value="0.0240"/>
-  <xacro:property name="prop_box_ixx"     value="0.01"/>
-  <xacro:property name="prop_box_iyy"     value="0.01"/>
-  <xacro:property name="prop_box_izz"     value="0.01"/>
+  <xacro:property name="prop_box_ixx"     value="0.00000425"/>
+  <xacro:property name="prop_box_iyy"     value="0.00010145"/>
+  <xacro:property name="prop_box_izz"     value="0.0001053"/>
   <xacro:property name="prop_box_length"    value="0.225"/>
   <xacro:property name="prop_box_width"     value="0.02"/>
