Commit message: [EDIT]: Adding Hexacopter as an SDF file

File: ros_ws/src/hexacopter_description/urdf/variable_tilt_hexacopter.urdf.xacro (robot description, xacro)
@@ -2,7 +2,7 @@
 <robot name="variable_tilt_hexacopter" xmlns:xacro="http://ros.org/wiki/xacro">
   <!-- ======================
-       1. Base Link
+       0. Properties
   ====================== -->
-  <!-- Base Dimensions and Parameters -->
+  <!-- Base -->
   <xacro:property name="base_mass"    value="1.5640"/>
   <xacro:property name="base_ixx"     value="0.00229686"/>
@@ -11,11 +11,189 @@
   <xacro:property name="base_radius"  value="0.071"/>
   <xacro:property name="base_length"  value="0.050"/>
-  <!-- Base Link -->
+  <!-- Landing Gear: Leg -->
+  <xacro:property name="gear_leg_mass"    value="0.1"/>
+  <xacro:property name="gear_leg_ixx"     value="0.0001"/>
+  <xacro:property name="gear_leg_iyy"     value="0.0001"/>
+  <xacro:property name="gear_leg_izz"     value="0.0001"/>
+  <xacro:property name="gear_leg_length"  value="0.1"/>
+  <xacro:property name="gear_leg_radius"  value="0.01"/>
+  <!-- Landing Gear: Skid -->
+  <xacro:property name="gear_skid_mass"       value="0.1"/>
+  <xacro:property name="gear_skid_ixx"        value="0.0001"/>
+  <xacro:property name="gear_skid_iyy"        value="0.0001"/>
+  <xacro:property name="gear_skid_izz"        value="0.0001"/>
+  <xacro:property name="gear_skid_length"     value="0.3"/>
+  <xacro:property name="gear_skid_width"      value="0.02"/>
+  <xacro:property name="gear_skid_thickness"  value="0.01"/>
+  <!-- Arm -->
+  <xacro:property name="arm_mass"    value="0.16"/>
+  <xacro:property name="arm_ixx"     value="0.000715213"/>
+  <xacro:property name="arm_iyy"     value="0.000715213"/>
+  <xacro:property name="arm_izz"     value="0.000032"/>
+  <xacro:property name="arm_length"  value="0.229"/>
+  <xacro:property name="arm_radius"  value="0.02"/>
+  <!-- Motor -->
+  <xacro:property name="motor_mass" value="0.0880"/>
+  <xacro:property name="motor_ixx"  value="0.000112917"/>
+  <xacro:property name="motor_iyy"  value="0.000112917"/>
+  <xacro:property name="motor_izz"  value="0.0000625"/>
+  <xacro:property name="motor_radius" value="0.02"/>
+  <xacro:property name="motor_height" value="0.05"/>
+  <!-- Propeller -->
+  <xacro:property name="prop_box_mass"    value="0.0240"/>
+  <xacro:property name="prop_box_ixx"     value="0.00000425"/>
+  <xacro:property name="prop_box_iyy"     value="0.00010145"/>
+  <xacro:property name="prop_box_izz"     value="0.0001053"/>
+  <xacro:property name="prop_box_length"    value="0.225"/>
+  <xacro:property name="prop_box_width"     value="0.02"/>
+  <xacro:property name="prop_box_thickness" value="0.01"/>
+  <xacro:property name="prop_offset_z"      value="0.02"/>
+  <!-- ======================
+       1. Macros
+  ====================== -->
+  <xacro:macro name="landing_gear" params="gear_name x y">
+    <link name="gear_leg_${gear_name}">
+      <inertial>
+        <mass value="${gear_leg_mass}"/>
+        <origin xyz="0 0 -${gear_leg_length/2}"/>
+        <inertia ixx="${gear_leg_ixx}" iyy="${gear_leg_iyy}" izz="${gear_leg_izz}" ixy="0" ixz="0" iyz="0"/>
+      </inertial>
+      <visual>
+        <origin xyz="0 0 -${gear_leg_length/2}"/>
+        <geometry>
+          <cylinder length="${gear_leg_length}" radius="${gear_leg_radius}"/>
+        </geometry>
+      </visual>
+      <collision>
+        <origin xyz="0 0 -${gear_leg_length/2}"/>
+        <geometry>
+          <cylinder length="${gear_leg_length}" radius="${gear_leg_radius}"/>
+        </geometry>
+      </collision>
+    </link>
+    <joint name="joint_gear_leg_${gear_name}" type="fixed">
+      <parent link="base"/>
+      <child link="gear_leg_${gear_name}"/>
+      <origin xyz="${x} ${y} 0"/>
+    </joint>
+    <link name="gear_skid_${gear_name}">
+      <inertial>
+        <mass value="${gear_skid_mass}"/>
+        <origin xyz="0 0 0"/>
+        <inertia ixx="${gear_skid_ixx}" iyy="${gear_skid_iyy}" izz="${gear_skid_izz}" ixy="0" ixz="0" iyz="0"/>
+      </inertial>
+      <visual>
+        <origin xyz="0 0 -${gear_leg_length}"/>
+        <geometry>
+          <box size="${gear_skid_length} ${gear_skid_width} ${gear_skid_thickness}"/>
+        </geometry>
+      </visual>
+      <collision>
+        <origin xyz="0 0 -${gear_leg_length}"/>
+        <geometry>
+          <box size="${gear_skid_length} ${gear_skid_width} ${gear_skid_thickness}"/>
+        </geometry>
+      </collision>
+    </link>
+    <joint name="joint_gear_skid_${gear_name}" type="fixed">
+      <parent link="gear_leg_${gear_name}"/>
+      <child link="gear_skid_${gear_name}"/>
+      <origin xyz="0 0 0"/>
+    </joint>
+  </xacro:macro>
+  <xacro:macro name="arm_motor" params="arm_name x y z rpy">
+    <link name="arm_${arm_name}">
+      <inertial>
+        <mass value="${arm_mass}"/>
+        <origin xyz="${arm_length * 0.5} 0 0"/>
+        <inertia ixx="${arm_ixx}" iyy="${arm_iyy}" izz="${arm_izz}" ixy="0" ixz="0" iyz="0"/>
+      </inertial>
+      <visual>
+        <origin xyz="0 0 0" rpy="0 1.5708 0"/>
+        <geometry>
+          <cylinder radius="${arm_radius}" length="${arm_length}"/>
+        </geometry>
+      </visual>
+      <collision>
+        <origin xyz="0 0 0" rpy="0 1.5708 0"/>
+        <geometry>
+          <cylinder radius="${arm_radius}" length="${arm_length}"/>
+        </geometry>
+      </collision>
+    </link>
+    <joint name="joint_arm_${arm_name}" type="revolute">
+      <parent link="base"/>
+      <child link="arm_${arm_name}"/>
+      <origin xyz="${x} ${y} ${z}" rpy="${rpy}"/>
+      <axis xyz="1 0 0"/>
+      <limit lower="-1.57" upper="1.57" effort="5" velocity="2.0"/>
+    </joint>
+    <link name="motor_${arm_name}">
+      <inertial>
+        <mass value="${motor_mass}"/>
+        <origin xyz="0 0 0"/>
+        <inertia ixx="${motor_ixx}" iyy="${motor_iyy}" izz="${motor_izz}" ixy="0" ixz="0" iyz="0"/>
+      </inertial>
+      <visual>
+        <origin xyz="0 0 0"/>
+        <geometry>
+          <cylinder radius="${motor_radius}" length="${motor_height}"/>
+        </geometry>
+      </visual>
+      <collision>
+        <origin xyz="0 0 0"/>
+        <geometry>
+          <cylinder radius="${motor_radius}" length="${motor_height}"/>
+        </geometry>
+      </collision>
+    </link>
+    <joint name="joint_motor_${arm_name}" type="fixed">
+      <parent link="arm_${arm_name}"/>
+      <child link="motor_${arm_name}"/>
+      <origin xyz="${arm_length/2 - motor_radius} 0 ${arm_radius}"/>
+    </joint>
+  </xacro:macro>
+  <xacro:macro name="propeller" params="prop_name motor_link">
+    <link name="prop_${prop_name}">
+      <inertial>
+        <mass value="${prop_box_mass}"/>
+        <origin xyz="0 0 ${prop_offset_z}"/>
+        <inertia ixx="${prop_box_ixx}" iyy="${prop_box_iyy}" izz="${prop_box_izz}" ixy="0" ixz="0" iyz="0"/>
+      </inertial>
+      <visual>
+        <origin xyz="0 0 ${prop_offset_z}"/>
+        <geometry>
+          <box size="${prop_box_length} ${prop_box_width} ${prop_box_thickness}"/>
+        </geometry>
+      </visual>
+      <collision>
+        <origin xyz="0 0 ${prop_offset_z}"/>
+        <geometry>
+          <box size="${prop_box_length} ${prop_box_width} ${prop_box_thickness}"/>
+        </geometry>
+      </collision>
+    </link>
+    <joint name="joint_prop_${prop_name}" type="continuous">
+      <parent link="${motor_link}"/>
+      <child link="prop_${prop_name}"/>
+      <axis xyz="0 0 1"/>
+    </joint>
+  </xacro:macro>
+  <!-- ======================
+       2. Link Definitions
+  ====================== -->
+  <!-- Dummy Root -->
+  <link name="base_dummy"/>
+  <joint name="joint_base_dummy_to_base" type="fixed">
+    <parent link="base_dummy"/>
+    <child link="base"/>
+    <origin xyz="0 0 0"/>
+  </joint>
+  <!-- Base -->
   <link name="base">
     <inertial>
       <mass value="${base_mass}"/>
       <origin xyz="0 0 0"/>
-      <inertia ixx="${base_ixx}" iyy="${base_iyy}" izz="${base_izz}"
-               ixy="0" ixz="0" iyz="0"/>
+      <inertia ixx="${base_ixx}" iyy="${base_iyy}" izz="${base_izz}" ixy="0" ixz="0" iyz="0"/>
     </inertial>
     <visual>
@@ -30,202 +208,15 @@
     </collision>
   </link>
-  <!-- ======================
-       2. Landing Gear
-  ====================== -->
-  <xacro:property name="gear_leg_mass"    value="0.1"/>
-  <xacro:property name="gear_leg_ixx"     value="0.0001"/>
-  <xacro:property name="gear_leg_iyy"     value="0.0001"/>
-  <xacro:property name="gear_leg_izz"     value="0.0001"/>
-  <xacro:property name="gear_leg_length"  value="0.1"/>
-  <xacro:property name="gear_leg_radius"  value="0.01"/>
-  <xacro:property name="gear_skid_mass"       value="0.1"/>
-  <xacro:property name="gear_skid_ixx"        value="0.0001"/>
-  <xacro:property name="gear_skid_iyy"        value="0.0001"/>
-  <xacro:property name="gear_skid_izz"        value="0.0001"/>
-  <xacro:property name="gear_skid_length"     value="0.3"/>
-  <xacro:property name="gear_skid_width"      value="0.02"/>
-  <xacro:property name="gear_skid_thickness"  value="0.01"/>
-  <xacro:macro name="landing_gear" params="gear_name x y">
-    <!-- Vertical leg link -->
-    <link name="gear_leg_${gear_name}">
-      <inertial>
-        <mass value="${gear_leg_mass}"/>
-        <origin xyz="0 0 -${gear_leg_length/2}"/>
-        <inertia ixx="${gear_leg_ixx}" iyy="${gear_leg_iyy}" izz="${gear_leg_izz}"
-                 ixy="0" ixz="0" iyz="0"/>
-      </inertial>
-      <visual>
-        <origin xyz="0 0 -${gear_leg_length/2}"/>
-        <geometry>
-          <cylinder length="${gear_leg_length}" radius="${gear_leg_radius}"/>
-        </geometry>
-      </visual>
-      <collision>
-        <origin xyz="0 0 -${gear_leg_length/2}"/>
-        <geometry>
-          <cylinder length="${gear_leg_length}" radius="${gear_leg_radius}"/>
-        </geometry>
-      </collision>
-    </link>
-    <joint name="joint_gear_leg_${gear_name}" type="fixed">
-      <parent link="base"/>
-      <child link="gear_leg_${gear_name}"/>
-      <origin xyz="${x} ${y} 0"/>
-    </joint>
-    <!-- Horizontal skid link -->
-    <link name="gear_skid_${gear_name}">
-      <inertial>
-        <mass value="${gear_skid_mass}"/>
-        <origin xyz="0 0 0"/>
-        <inertia ixx="${gear_skid_ixx}" iyy="${gear_skid_iyy}" izz="${gear_skid_izz}"
-                 ixy="0" ixz="0" iyz="0"/>
-      </inertial>
-      <visual>
-        <origin xyz="0 0 -${gear_leg_length}"/>
-        <geometry>
-          <box size="${gear_skid_length} ${gear_skid_width} ${gear_skid_thickness}"/>
-        </geometry>
-      </visual>
-      <collision>
-        <origin xyz="0 0 -${gear_leg_length}"/>
-        <geometry>
-          <box size="${gear_skid_length} ${gear_skid_width} ${gear_skid_thickness}"/>
-        </geometry>
-      </collision>
-    </link>
-    <joint name="joint_gear_skid_${gear_name}" type="fixed">
-      <parent link="gear_leg_${gear_name}"/>
-      <child link="gear_skid_${gear_name}"/>
-      <origin xyz="0 0 0"/>
-    </joint>
-  </xacro:macro>
-  <!-- Define left and right landing gears -->
+  <!-- Landing Gear -->
   <xacro:landing_gear gear_name="left"  x="0"  y="0.05"/>
   <xacro:landing_gear gear_name="right" x="0"  y="-0.05"/>
-  <!-- ======================
-       3. Arm + Motor Properties
-  ====================== -->
-  <xacro:property name="arm_mass"    value="0.16"/>
-  <xacro:property name="arm_ixx"     value="0.000715213"/>
-  <xacro:property name="arm_iyy"     value="0.000715213"/>
-  <xacro:property name="arm_izz"     value="0.000032"/>
-  <xacro:property name="arm_length"  value="0.229"/>
-  <xacro:property name="arm_radius"  value="0.02"/>
-  <xacro:property name="motor_mass" value="0.0880"/>
-  <xacro:property name="motor_ixx"  value="0.000112917"/>
-  <xacro:property name="motor_iyy"  value="0.000112917"/>
-  <xacro:property name="motor_izz"  value="0.0000625"/>
-  <xacro:property name="motor_radius" value="0.02"/>
-  <xacro:property name="motor_height" value="0.05"/>
-  <xacro:property name="prop_box_mass"    value="0.0240"/>
-  <xacro:property name="prop_box_ixx"     value="0.00000425"/>
-  <xacro:property name="prop_box_iyy"     value="0.00010145"/>
-  <xacro:property name="prop_box_izz"     value="0.0001053"/>
-  <xacro:property name="prop_box_length"    value="0.225"/>
-  <xacro:property name="prop_box_width"     value="0.02"/>
-  <xacro:property name="prop_box_thickness" value="0.01"/>
-  <xacro:property name="prop_offset_z"      value="0.02"/>
-  <!-- ======================
-       4. Macro: Arm + Motor
-  ====================== -->
-  <xacro:macro name="arm_motor" params="arm_name x y z rpy">
-    <link name="arm_${arm_name}">
-      <inertial>
-        <mass value="${arm_mass}"/>
-        <origin xyz="${arm_length * 0.5} 0 0"/>
-        <inertia ixx="${arm_ixx}" iyy="${arm_iyy}" izz="${arm_izz}"
-                 ixy="0" ixz="0" iyz="0"/>
-      </inertial>
-      <visual>
-        <origin xyz="0 0 0" rpy="0 1.5708 0"/>
-        <geometry>
-          <cylinder radius="${arm_radius}" length="${arm_length}"/>
-        </geometry>
-      </visual>
-      <collision>
-        <origin xyz="0 0 0" rpy="0 1.5708 0"/>
-        <geometry>
-          <cylinder radius="${arm_radius}" length="${arm_length}"/>
-        </geometry>
-      </collision>
-    </link>
-    <!-- Revolute joint to allow arm to rotate for tilt -->
-    <joint name="joint_arm_${arm_name}" type="revolute">
-      <parent link="base"/>
-      <child link="arm_${arm_name}"/>
-      <origin xyz="${x} ${y} ${z}" rpy="${rpy}"/>
-      <axis xyz="1 0 0"/>
-      <limit lower="-1.57" upper="1.57" effort="5" velocity="2.0"/>
-    </joint>
-    <!-- Motor (Fixed to Arm) -->
-    <link name="motor_${arm_name}">
-      <inertial>
-        <mass value="${motor_mass}"/>
-        <origin xyz="0 0 0"/>
-        <inertia ixx="${motor_ixx}" iyy="${motor_iyy}" izz="${motor_izz}"
-                 ixy="0" ixz="0" iyz="0"/>
-      </inertial>
-      <visual>
-        <origin xyz="0 0 0"/>
-        <geometry>
-          <cylinder radius="${motor_radius}" length="${motor_height}"/>
-        </geometry>
-      </visual>
-      <collision>
-        <origin xyz="0 0 0"/>
-        <geometry>
-          <cylinder radius="${motor_radius}" length="${motor_height}"/>
-        </geometry>
-      </collision>
-    </link>
-    <!-- Fixed motor joint (no rotation with arm) -->
-    <joint name="joint_motor_${arm_name}" type="fixed">
-      <parent link="arm_${arm_name}"/>
-      <child link="motor_${arm_name}"/>
-      <origin xyz="${arm_length/2 - motor_radius} 0 ${arm_radius}"/>
-    </joint>
-  </xacro:macro>
-  <!-- ======================
-       5. Macro: Propeller
-  ====================== -->
-  <xacro:macro name="propeller" params="prop_name motor_link">
-    <link name="prop_${prop_name}">
-      <inertial>
-        <mass value="${prop_box_mass}"/>
-        <origin xyz="0 0 ${prop_offset_z}"/>
-        <inertia ixx="${prop_box_ixx}" iyy="${prop_box_iyy}" izz="${prop_box_izz}"
-                 ixy="0" ixz="0" iyz="0"/>
-      </inertial>
-      <visual>
-        <origin xyz="0 0 ${prop_offset_z}"/>
-        <geometry>
-          <box size="${prop_box_length} ${prop_box_width} ${prop_box_thickness}"/>
-        </geometry>
-      </visual>
-      <collision>
-        <origin xyz="0 0 ${prop_offset_z}"/>
-        <geometry>
-          <box size="${prop_box_length} ${prop_box_width} ${prop_box_thickness}"/>
-        </geometry>
-      </collision>
-    </link>
-    <joint name="joint_prop_${prop_name}" type="continuous">
-      <parent link="${motor_link}"/>
-      <child link="prop_${prop_name}"/>
-      <axis xyz="0 0 1"/>
-    </joint>
-  </xacro:macro>
-  <!-- ======================
-       6. Define 6 Arms + Motors
-  ====================== -->
-  <xacro:arm_motor arm_name="1" x="${arm_length/2 + base_radius}"      y="0"    z="0" rpy="0 0 0"/>
+  <!-- Arms -->
+  <xacro:arm_motor arm_name="1" x="${arm_length/2 + base_radius}" y="0" z="0" rpy="0 0 0"/>
   <xacro:arm_motor arm_name="2" x="${(arm_length/2 + base_radius)*0.5}" y="${0.866 * (arm_length/2 + base_radius)}" z="0" rpy="0 0 1.047"/>
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
Commit message: [EDIT]: Updating the Xacro and SDF files with more correct configurations.

File: ros_ws/src/hexacopter_description/urdf/variable_tilt_hexacopter.urdf.xacro (robot description, xacro)
@@ -227,10 +227,16 @@
   <!-- Pluggins -->
   <!-- Pose Publisher Plugin -->
-    <plugin filename="ignition-gazebo-pose-publisher-system"
-            name="ignition::gazebo::systems::PosePublisher">
-      <publish_link_pose>true</publish_link_pose>
+  <plugin filename="ignition-gazebo-pose-publisher-system" name="ignition::gazebo::systems::PosePublisher">
+    <publish_link_pose>true</publish_link_pose>
       <publish_sensor_pose>true</publish_sensor_pose>
-    </plugin>
-    <!-- Joint states plugin -->
+      <publish_collision_pose>false</publish_collision_pose>
+      <publish_visual_pose>false</publish_visual_pose>
+      <publish_nested_model_pose>true</publish_nested_model_pose>
+      <publish_model_pose>false</publish_model_pose>
+      <use_pose_vector_msg>true</use_pose_vector_msg>
+      <static_publisher>true</static_publisher>
+      <static_update_frequency>100</static_update_frequency>
+  </plugin>
+  <!-- Joint states plugin -->
     <plugin
       filename="ignition-gazebo-joint-state-publisher-system"
@@ -241,11 +247,10 @@
     <plugin filename="ignition-gazebo-imu-system"
             name="ignition::gazebo::systems::Imu">
-      <topic>/hexacopter/imu</topic>
-      <link_name>base</link_name>
     </plugin>
     <!-- Odometry Plugin -->
     <plugin filename="ignition-gazebo-odometry-publisher-system"
             name="ignition::gazebo::systems::OdometryPublisher">
-      <topic>/hexacopter/odom</topic>
+      <dimensions>3</dimensions>
+      <odom_publish_frequency>100</odom_publish_frequency>
     </plugin>
     <!-- ========== Sub-macros ========== -->
@@ -272,24 +277,4 @@
       </plugin>
     </xacro:macro>
-    <!-- Lift and drag plugin -->
-    <xacro:macro name="lift_drag_plugin" params="blade_id link_name upward_x upward_y">
-      <plugin filename="libignition-gazebo-lift-drag-system"
-              name="ignition::gazebo::systems::LiftDrag">
-        <a0>0.2</a0>
-        <cla>10.0</cla>
-        <cda>0.0001</cda>
-        <cma>0.00</cma>
-        <alpha_stall>10.0</alpha_stall>
-        <cla_stall>1.0</cla_stall>
-        <cda_stall>0.001</cda_stall>
-        <cma_stall>0.0</cma_stall>
-        <cp>${prop_box_length/2} 0 0</cp>
-        <area>${prop_box_length * prop_box_width}</area>
-        <air_density>1.2041</air_density>
-        <forward>0 0 -1</forward>
-        <upward>${upward_x} ${upward_y} 0</upward>
-        <link_name>${link_name}</link_name>
-      </plugin>
-    </xacro:macro>
     <!-- Joint controller plugin -->
     <xacro:macro name="joint_controller_plugin" params="joint">
@@ -302,17 +287,10 @@
     <!-- ========== Plugin Instantiations ========== -->
     <!-- Motor plugins -->
-    <xacro:motor_plugin id="1" joint="joint_prop_1" link="prop_1" direction="ccw"/>
-    <xacro:motor_plugin id="2" joint="joint_prop_2" link="prop_2" direction="cw"/>
-    <xacro:motor_plugin id="3" joint="joint_prop_3" link="prop_3" direction="ccw"/>
-    <xacro:motor_plugin id="4" joint="joint_prop_4" link="prop_4" direction="cw"/>
-    <xacro:motor_plugin id="5" joint="joint_prop_5" link="prop_5" direction="ccw"/>
-    <xacro:motor_plugin id="6" joint="joint_prop_6" link="prop_6" direction="cw"/>
-    <!-- Lift-drag plugins -->
-    <xacro:lift_drag_plugin blade_id="1" link_name="prop_1" upward_x="0.0" upward_y="1.0" />
-    <xacro:lift_drag_plugin blade_id="2" link_name="prop_2" upward_x="0.866" upward_y="-0.5" />
-    <xacro:lift_drag_plugin blade_id="3" link_name="prop_3" upward_x="-0.866" upward_y="-0.5" />
-    <xacro:lift_drag_plugin blade_id="4" link_name="prop_4" upward_x="0.0" upward_y="-1.0" />
-    <xacro:lift_drag_plugin blade_id="5" link_name="prop_5" upward_x="0.866" upward_y="0.5" />
-    <xacro:lift_drag_plugin blade_id="6" link_name="prop_6" upward_x="-0.866" upward_y="0.5" />
+    <xacro:motor_plugin id="0" joint="joint_prop_1" link="prop_1" direction="ccw"/>
+    <xacro:motor_plugin id="1" joint="joint_prop_2" link="prop_2" direction="cw"/>
+    <xacro:motor_plugin id="2" joint="joint_prop_3" link="prop_3" direction="ccw"/>
+    <xacro:motor_plugin id="3" joint="joint_prop_4" link="prop_4" direction="cw"/>
+    <xacro:motor_plugin id="4" joint="joint_prop_5" link="prop_5" direction="ccw"/>
+    <xacro:motor_plugin id="5" joint="joint_prop_6" link="prop_6" direction="cw"/>
     <!-- Joint controllers -->
     <xacro:joint_controller_plugin joint="joint_arm_1"/>
