Commit message: [EDIT]: Tidy ups.

File: ros_ws/src/hexacopter_description/urdf/variable_tilt_hexacopter.urdf (robot description, URDF)
Before this commit: robot variable_tilt_hexacopter, 24 links, 23 joints
Links:
- added link camera_link; visual box ; visual cylinder 
Joints:
- added joint camera_joint: type fixed, parent base, child camera_link, origin xyz=0.0 0.0 0.025

File: ros_ws/src/hexacopter_description/urdf/variable_tilt_hexacopter.urdf.xacro (robot description, xacro)
@@ -295,5 +295,5 @@
       <always_on>true</always_on>
       <update_rate>30.0</update_rate>
-      <pose>0.05 0 0 0 0 0</pose> <!-- Slight x offset from IMU -->
+      <pose>0 0 0.025 0 0 0</pose> <!-- Slight x offset from IMU -->
       <camera>
         <horizontal_fov>1.3962634</horizontal_fov>
@@ -317,4 +317,73 @@
     </sensor>
   </link>
+  <!-- Camera Link -->
+  <link name="camera_link">
+    <inertial>
+      <pose>0.0 0.0 0.0 0 0 0</pose>
+      <mass>0.050</mass>
+      <inertia>
+        <ixx>0.00004</ixx>
+        <ixy>0</ixy>
+        <ixz>0</ixz>
+        <iyy>0.00004</iyy>
+        <iyz>0</iyz>
+        <izz>0.00004</izz>
+      </inertia>
+    </inertial>
+    <visual name="mono_cam/visual/housing">
+      <geometry>
+        <box>
+          <size>0.02 0.04 0.04</size>
+        </box>
+      </geometry>
+    </visual>
+    <visual name="mono_cam/visual/lens">
+      <pose>0.015 0 0 0 1.5707 0</pose>
+      <geometry>
+        <cylinder>
+          <radius>0.008</radius>
+          <length>0.01</length>
+        </cylinder>
+      </geometry>
+    </visual>
+    <visual name="mono_cam/visual/lens_glass">
+      <pose>0.014 0 0 0 0 0</pose>
+      <geometry>
+        <sphere>
+          <radius>0.0079</radius>
+        </sphere>
+      </geometry>
+      <material>
+        <ambient>.4 .4 .5 .95</ambient>
+        <diffuse>.4 .4 .5 .95</diffuse>
+        <specular>1 1 1 1</specular>
+        <emissive>0 0 0 1</emissive>
+      </material>
+    </visual>
+    <sensor name="imager" type="camera">
+      <pose>0 0 0 0 0 0</pose>
+      <camera>
+        <horizontal_fov>1.74</horizontal_fov>
+        <image>
+          <width>1280</width>
+          <height>960</height>
+        </image>
+        <clip>
+          <near>0.1</near>
+          <far>3000</far>
+        </clip>
+      </camera>
+      <always_on>1</always_on>
+      <update_rate>30</update_rate>
+      <visualize>true</visualize>
+    </sensor>
+    <gravity>true</gravity>
+    <velocity_decay/>
+  </link>
+  <joint name="camera_joint" type="fixed">
+    <parent link="base"/>
+    <child link="camera_link"/>
+    <origin xyz="0.0 0.0 0.025"/>
+  </joint>
   <!-- Landing Gear -->
   <xacro:landing_gear gear_name="left"  x="0"  y="0.05"/>
@@ -370,6 +439,6 @@
         <timeConstantUp>0.0125</timeConstantUp>
         <timeConstantDown>0.025</timeConstantDown>
-        <maxRotVelocity>800.0</maxRotVelocity>
-        <motorConstant>0.000918</motorConstant>
+        <maxRotVelocity>1000.0</maxRotVelocity>
+        <motorConstant>8.54858e-06</motorConstant>
         <momentConstant>0.016</momentConstant>
         <commandSubTopic>command/motor_speed</commandSubTopic>
